File: CANT_Shield/CANT.sch (KiCad schematic (older format))
At the start: 13 parts, among them CN7 CN7, CN8 CN8, J1 Screw_Terminal_01x02, U1 SN65HVD232, U2 74LVC1G66

Commit message: Changed to rev 0.2, switched to using TJA1051 CAN transceiver
Parts:
- removed U1: SN65HVD232, Housings_SOIC:SOIC-8_3.9x4.9mm_Pitch1.27mm, symbol CANT-rescue:SN65HVD232
- added C6: 0.1uF, Capacitors_SMD:C_0805_HandSoldering, symbol CANT-rescue:C_Small
- added U1: TJA1051T_3, Housings_SOIC:SOIC-8_3.9x4.9mm_Pitch1.27mm, symbol TJA1051:TJA1051T_3
Connections:
- net labels added: 5V
- wire segments 56 -> 64
- no-connect marks 30 -> 29
Other:
- moved on the sheet: C1, C2, C3
Changed lines of the file:
@@
-	1    0    0    -1
-$EndComp
-$Comp
-L CANT-rescue:SN65HVD232 U1
-U 1 1 5A7C753C
-P 3350 2550
-F 0 "U1" H 3250 2950 50  0000 R CNN
-F 1 "SN65HVD232" H 3250 2850 50  0000 R CNN
-F 2 "Housings_SOIC:SOIC-8_3.9x4.9mm_Pitch1.27mm" H 3350 2050 50  0001 C CNN
-F 3 "" H 3250 2950 50  0001 C CNN
-	1    3350 2550
 	1    0    0    -1
 $EndComp
 NoConn ~ 1350 2550
-$Comp
-L CANT-rescue:VCC #PWR01
-U 1 1 5A7C7FEA
-P 3350 1650
-F 0 "#PWR01" H 3350 1500 50  0001 C CNN
-F 1 "VCC" H 3350 1800 50  0000 C CNN
-F 2 "" H 3350 1650 50  0001 C CNN
-F 3 "" H 3350 1650 50  0001 C CNN
-	1    3350 1650
-	1    0    0    -1
-$EndComp
 $Comp
 L CANT-rescue:GND #PWR02
 U 1 1 5A7C812E
-P 3350 3200
-F 0 "#PWR02" H 3350 2950 50  0001 C CNN
-F 1 "GND" H 3350 3050 50  0000 C CNN
-F 2 "" H 3350 3200 50  0001 C CNN
-F 3 "" H 3350 3200 50  0001 C CNN
-	1    3350 3200
+P 3050 3150
+F 0 "#PWR02" H 3050 2900 50  0001 C CNN
+F 1 "GND" H 3050 3000 50  0000 C CNN
+F 2 "" H 3050 3150 50  0001 C CNN
+F 3 "" H 3050 3150 50  0001 C CNN
+	1    3050 3150
 	1    0    0    -1
 $EndComp
@@
 L CANT-rescue:GND #PWR03
 U 1 1 5A7C925A
-P 2750 1750
-F 0 "#PWR03" H 2750 1500 50  0001 C CNN
-F 1 "GND" H 2750 1600 50  0000 C CNN
-F 2 "" H 2750 1750 50  0001 C CNN
-F 3 "" H 2750 1750 50  0001 C CNN
-	1    2750 1750
+P 2400 1800
+F 0 "#PWR03" H 2400 1550 50  0001 C CNN
+F 1 "GND" H 2400 1650 50  0000 C CNN
+F 2 "" H 2400 1800 50  0001 C CNN
+F 3 "" H 2400 1800 50  0001 C CNN
+	1    2400 1800
 	0    1    1    0
 $EndComp
@@
 L CANT-rescue:GND #PWR04
 U 1 1 5A7C927A
-P 2750 2000
-F 0 "#PWR04" H 2750 1750 50  0001 C CNN
-F 1 "GND" H 2750 1850 50  0000 C CNN
-F 2 "" H 2750 2000 50  0001 C CNN
-F 3 "" H 2750 2000 50  0001 C CNN
-	1    2750 2000
+P 2400 2050
+F 0 "#PWR04" H 2400 1800 50  0001 C CNN
+F 1 "GND" H 2400 1900 50  0000 C CNN
+F 2 "" H 2400 2050 50  0001 C CNN
+F 3 "" H 2400 2050 50  0001 C CNN
+	1    2400 2050
 	0    1    1    0
 $EndComp
@@
 L CANT-rescue:C_Small C2
 U 1 1 5A7C92BE
-P 3000 1750
-F 0 "C2" H 3010 1820 50  0000 L CNN
-F 1 "0.1uF" H 2750 1650 50  0000 L CNN
-F 2 "Capacitors_SMD:C_0805_HandSoldering" H 3000 1750 50  0001 C CNN
-F 3 "" H 3000 1750 50  0001 C CNN
-	1    3000 1750
+P 2650 1800
+F 0 "C2" H 2660 1870 50  0000 L CNN
+F 1 "0.1uF" H 2400 1700 50  0000 L CNN
+F 2 "Capacitors_SMD:C_0805_HandSoldering" H 2650 1800 50  0001 C CNN
+F 3 "" H 2650 1800 50  0001 C CNN
+	1    2650 1800
 	0    1    1    0
 $EndComp
@@
 L CANT-rescue:C_Small C3
 U 1 1 5A7C9304
-P 3000 2000
-F 0 "C3" H 3010 2070 50  0000 L CNN
-F 1 "10 uF" H 2900 1900 50  0000 L CNN
-F 2 "Capacitors_SMD:C_0805_HandSoldering" H 3000 2000 50  0001 C CNN
-F 3 "" H 3000 2000 50  0001 C CNN
-	1    3000 2000
+P 2650 2050
+F 0 "C3" H 2660 2120 50  0000 L CNN
+F 1 "10 uF" H 2550 1950 50  0000 L CNN
+F 2 "Capacitors_SMD:C_0805_HandSoldering" H 2650 2050 50  0001 C CNN
+F 3 "" H 2650 2050 50  0001 C CNN
+	1    2650 2050
 	0    1    1    0
 $EndComp
@@
 NoConn ~ 1350 2650
 NoConn ~ 1350 2750
-NoConn ~ 1350 2950
 NoConn ~ 1350 3250
 NoConn ~ 1850 3250
@@
 Text GLabel 6300 2500 0    60   Input ~ 0
 CAN_RX
-Text GLabel 2700 2450 0    60   Input ~ 0
+Text GLabel 2400 2400 0    60   Input ~ 0
 CAN_TX
-Text GLabel 2700 2550 0    60   Input ~ 0
+Text GLabel 2400 2500 0    60   Input ~ 0
 CAN_RX
 Wire Wire Line
-	3350 2950 3350 3150
-Wire Wire Line
 	4150 2050 4150 1950
 Wire Wire Line
-	3350 2250 3350 2000
-Wire Wire Line
-	3100 1750 3350 1750
-Connection ~ 3350 1750
-Wire Wire Line
-	3100 2000 3350 2000
-Connection ~ 3350 2000
-Wire Wire Line
-	2900 2000 2750 2000
-Wire Wire Line
-	2900 1750 2750 1750
+	2750 2050 3000 2050
+Wire Wire Line
+	2550 2050 2400 2050
 Wire Wire Line
 	3800 1950 3850 1950
 Wire Wire Line
-	4750 2650 3750 2650
-Wire Wire Line
-	3800 2550 3750 2550
-Connection ~ 4750 2050
-Wire Wire Line
-	3800 1100 3800 1950
-Wire Wire Line
 	4750 1200 4750 2050
 Wire Wire Line
@@
 Wire Wire Line
 	3800 1100 4950 1100
-Connection ~ 3800 1950
 Wire Wire Line
 	6250 2000 6300 2000
@@
 	6800 2500 6300 2500
 Wire Wire Line
-	2700 2450 2850 2450
-Wire Wire Line
-	2950 2550 2700 2550
+	2400 2400 2550 2400
 $Comp
 L CANT-rescue:C_Small C1
 U 1 1 5A7CBB90
-P 2850 2950
-F 0 "C1" H 2860 3020 50  0000 L CNN
-F 1 "100pF" H 2860 2870 50  0000 L CNN
-F 2 "Capacitors_SMD:C_0805_HandSoldering" H 2850 2950 50  0001 C CNN
-F 3 "" H 2850 2950 50  0001 C CNN
-	1    2850 2950
-	1    0    0    -1
-$EndComp
-Wire Wire Line
-	2850 2450 2850 2850
-Connection ~ 2850 2450
-Wire Wire Line
-	2850 3050 2850 3150
-Wire Wire Line
-	2850 3150 3350 3150
-Connection ~ 3350 3150
+P 2550 2900
+F 0 "C1" H 2560 2970 50  0000 L CNN
+F 1 "100pF" H 2560 2820 50  0000 L CNN
+F 2 "Capacitors_SMD:C_0805_HandSoldering" H 2550 2900 50  0001 C CNN
+F 3 "" H 2550 2900 50  0001 C CNN
+	1    2550 2900
+	1    0    0    -1
+$EndComp
+Wire Wire Line
+	2550 2400 2550 2800
+Wire Wire Line
+	2550 3000 2550 3100
+Wire Wire Line
+	2550 3100 2800 3100
 $Comp
 L CANT-rescue:PWR_FLAG #FLG010
@@
 $EndComp
 Wire Wire Line
-	3350 1750 3350 1650
-Wire Wire Line
-	3350 2000 3350 1750
-Wire Wire Line
-	4750 2050 4750 2650
-Wire Wire Line
-	3800 1950 3800 2550
+	3000 2050 3000 1800
 Wire Wire Line
 	6300 2000 6350 2000
@@
 	1050 3100 1050 3150
 Wire Wire Line
-	2850 2450 2950 2450
-Wire Wire Line
-	3350 3150 3350 3200
+	3050 3100 3050 3150
 Wire Wire Line
 	1100 3150 1350 3150
@@
 Wire Wire Line
 	7900 2600 7300 2600
+$Comp
+L TJA1051:TJA1051T_3 U1
+U 1 1 5B4D3873
+P 3300 2600
+F 0 "U1" H 3300 3178 50  0000 C CNN
+F 1 "TJA1051T_3" H 3300 3087 50  0000 C CNN
+F 2 "Housings_SOIC:SOIC-8_3.9x4.9mm_Pitch1.27mm" H 3300 2100 50  0001 C CIN
+F 3 "" H 3300 2600 50  0001 C CNN
+	1    3300 2600
+	1    0    0    -1
+$EndComp
+Wire Wire Line
+	3800 1100 3800 1950
+Wire Wire Line
+	2800 2400 2550 2400
+Connection ~ 2550 2400
+Wire Wire Line
+	2400 2500 2800 2500
+Wire Wire Line
+	3800 2500 3800 1950
+Connection ~ 3800 1950
+Wire Wire Line
+	3800 2700 4750 2700
+Wire Wire Line
+	4750 2700 4750 2050
+Connection ~ 4750 2050
+Wire Wire Line
+	3300 3000 3300 3100
+Wire Wire Line
+	3300 3100 3050 3100
+Connection ~ 3050 3100
+Wire Wire Line
+	2800 2800 2800 3100
+Connection ~ 2800 3100
+Wire Wire Line
+	2800 3100 3050 3100
+Text GLabel 1050 2950 0    50   Input ~ 0
+5V
+Wire Wire Line
+	1350 2950 1050 2950
+Text GLabel 3000 1550 0    50   Input ~ 0
+5V
+Wire Wire Line
+	3000 1550 3000 1800
+Connection ~ 3000 1800
+Wire Wire Line
+	3000 2050 3000 2200
+Wire Wire Line
+	3000 2200 3300 2200
+Connection ~ 3000 2050
+$Comp
+L CANT-rescue:VCC #PWR01
+U 1 1 5B4EEA50
+P 2250 2700
+F 0 "#PWR01" H 2250 2550 50  0001 C CNN
+F 1 "VCC" V 2268 2827 50  0000 L CNN
+F 2 "" H 2250 2700 50  0001 C CNN
+F 3 "" H 2250 2700 50  0001 C CNN
+	1    2250 2700
+	0    -1   -1   0
+$EndComp
+Wire Wire Line
+	2250 2700 2800 2700
+Wire Wire Line
+	2550 1800 2400 1800
+Wire Wire Line
+	2750 1800 3000 1800
+$Comp
+L CANT-rescue:C_Small C6
+U 1 1 5B4F4D4E
+P 2250 2900
+F 0 "C6" H 2260 2970 50  0000 L CNN
+F 1 "0.1uF" H 2000 2800 50  0000 L CNN
+F 2 "Capacitors_SMD:C_0805_HandSoldering" H 2250 2900 50  0001 C CNN
+F 3 "" H 2250 2900 50  0001 C CNN
+	1    2250 2900
+	-1   0    0    1
+$EndComp
+Wire Wire Line
+	2250 2700 2250 2800
+Connection ~ 2250 2700
+Wire Wire Line
+	2250 3000 2250 3100
+Wire Wire Line
+	2250 3100 2550 3100
+Connection ~ 2550 3100
 $EndSCHEMATC
