File: CANTboard/CANT.kicad_pcb (KiCad board)
At the start: 2 copper layers, 67.8 x 45.5 mm, 49 parts, among them J1 Screw_Terminal_01x04, J2 Conn_02x08_Odd_Even, P1 SWD, P3 USB, SW1 SW_SPST, U1 STM32H743VITx, U2 MCP2558FD-xSN, U3 LD1117S33TR, U4 74LVC1G66, U5 74LVC1G66, U6 MCP2558FD-xSN, U7 USBLC6-2SC6, Y1 Crystal

Commit message: Finished layout, ordered first set of prototype boards
Parts:
- removed the C3 at (118.7, 79.8)
- removed the C6 at (97.0, 92.2)
- removed the C9 at (118.6, 83.8)
- removed the R1 at (80.0, 72.4)
- removed the R2 at (137.7, 101.3)
- removed the U4 at (84.3, 84.1)
- removed the U7 at (97.0, 75.7)
- added C10: 100nF, Capacitor_SMD:C_0805_2012Metric, F.Cu at (118.6, 80.8)
- added C11: 10uF, Capacitor_SMD:C_0805_2012Metric, F.Cu at (116.2, 73.9)
- added C12: 2.2uF, Capacitor_SMD:C_0805_2012Metric, F.Cu at (102.6, 114.6)
- added C14: 2.2uF, Capacitor_SMD:C_0805_2012Metric, F.Cu at (118.6, 82.8)
- added C2: 100nF, Capacitor_SMD:C_0805_2012Metric, F.Cu at (114.3, 114.3)
- added C22: 100nF, Capacitor_SMD:C_0805_2012Metric, F.Cu at (94.5, 91.2)
- added C4: 4.7uF, Capacitor_SMD:C_0805_2012Metric, F.Cu at (118.6, 78.6)
- added G***: LOGO, KiCad:Logo, B.Cu at (115.3, 89.7)
- added J2: Screw_Terminal_01x02, TerminalBlock_Phoenix:TerminalBlock_Phoenix_PT-1,5-2-3.5-H_1x02_P3.50mm_Horizontal, F.Cu at (91.9, 114.2)
- added R11: 120, Resistor_SMD:R_0805_2012Metric, F.Cu at (80.1, 72.1)
- added R13: 10k, Resistor_SMD:R_0805_2012Metric, F.Cu at (127.8, 104.5)
- added R4: 4.7K, Resistor_SMD:R_0805_2012Metric, F.Cu at (107.6, 114.4)
- added R5: 4.7K, Resistor_SMD:R_0805_2012Metric, F.Cu at (107.7, 110.4)
- added R7: 47, Resistor_SMD:R_0805_2012Metric, F.Cu at (96.0, 109.3)
- added R8: 47, Resistor_SMD:R_0805_2012Metric, F.Cu at (96.0, 107.2)
- added U1: USBLC6-2SC6, Package_TO_SOT_SMD:SOT-23-6, F.Cu at (107.1, 75.4)
- added U2: SN74LVC1G14DBV, Package_TO_SOT_SMD:SOT-23-5, F.Cu at (121.2, 110.7)
- added U3: ST485EBDR, Package_SO:SOIC-8_3.9x4.9mm_P1.27mm, F.Cu at (114.0, 110.1)
- added U9: 74LVC1G66, Package_TO_SOT_SMD:SOT-353_SC-70-5_Handsoldering, F.Cu at (82.5, 76.8)
- C13: value 100nF -> 2.2uF
- C8: value 10uF -> 100nF
- moved C8 42.7 mm to (124.2, 114.3), turned to 0 degrees
- moved P2 33.6 mm to (137.5, 103.5)
- moved C13 32.8 mm to (102.6, 110.4), turned to 270 degrees
- moved R6 18.1 mm to (129.7, 113.5), turned to 0 degrees
- moved R10 17.9 mm to (86.2, 112.0), turned to 270 degrees
- moved SW1 16.3 mm to (135.0, 72.6)
- moved U7 15.0 mm to (83.7, 106.4), turned to 270 degrees
- moved JP3 14.6 mm to (123.3, 101.1), turned to 0 degrees
- moved C7 12.4 mm to (116.2, 69.3)
- moved C18 12.3 mm to (129.5, 108.7), turned to 0 degrees
- moved D2 9.40 mm to (94.2, 69.0)
- moved R9 9.34 mm to (80.9, 112.1), turned to 90 degrees
- moved F1 8.99 mm to (111.3, 69.2)
- moved R12 8.93 mm to (85.2, 72.1), turned to 90 degrees
- moved P1 8.75 mm to (104.0, 69.1)
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- renumbered C10 to C15, C18 to C16, C19 to C17, C20 to C18, C14 to C19, C15 to C20, C5 to C21, C16 to C23, C17 to C24, C2 to C3, C4 to C5, C11 to C6, C12 to C9, J2 to J1, J1 to J3, JP3 to JP1, JP1 to JP3, P3 to P1, P1 to P2, R3 to R1, R7 to R10, R5 to R12, R4 to R2, R8 to R3, R9 to R6, R6 to R9, U3 to U4, U1 to U5, U2 to U6, U5 to U7, U6 to U8
Connections:
- C13 pad 1: VCC -> GND
- C13 pad 2: GND -> Net-(C13-Pad2)
- U5 pad 22: Net-(U1-Pad22) -> J1708_TX
- U5 pad 23: Net-(U1-Pad23) -> J1708_RX
Routing:
- net GND: track 0.00 -> 117.1 mm
- net /NRST: track 0.00 -> 99.4 mm, vias 0 -> 1
- net VBUS: track 0.00 -> 85.9 mm, vias 0 -> 4
- net VCC: track 0.00 -> 73.8 mm, vias 0 -> 15
- net /SWDIO: track 0.00 -> 48.1 mm, vias 0 -> 1
- net /SWCLK: track 0.00 -> 47.9 mm, vias 0 -> 1
- net LED_ACT2: track 0.00 -> 42.1 mm, vias 0 -> 4
- net CAN2_L: track 0.00 -> 39.8 mm, vias 0 -> 2
- net LED_ACT1: track 0.00 -> 38.3 mm, vias 0 -> 2
- net CAN2_SHORT: track 0.00 -> 35.7 mm, vias 0 -> 2
- net BOOT0: track 0.00 -> 33.8 mm, vias 0 -> 1
- net CAN2_H: track 0.00 -> 32.0 mm
- net CAN1_SHORT: track 0.00 -> 30.3 mm, vias 0 -> 2
- net LED_PWR1: track 0.00 -> 28.3 mm, vias 0 -> 2
- net J1708_RX: track 0.00 -> 23.4 mm
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Other:
- board size 67.8 x 45.5 mm -> 67.6 x 50.8 mm
- board text added: "+"
- board text added: "-"
- board text added: "100K"
- board text added: "100nF"
- board text added: "10K"
- board text added: "10uF"
- board text added: "120"
- board text added: "1uF"
- board text added: "2.2uF"
- board text added: "26pF"
- board text added: "4.7K"
- board text added: "4.7uF"
- board text added: "47"
- board text added: "68"
- board text added: "BOOT"
- board text added: "CANT"
- board text added: "CLK"
- board text added: "CanCat"
- board text added: "DIO"
- board text added: "GND"
- board text added: "J1708"
- board text added: "NRST"
- board text added: "One Board To Run Them All https://github.com/bitbane/CANT @b1tbane"
- board text added: "PWR"
- board text added: "Prog1"
- board text added: "Prog2"
- board text added: "Prog3"
- board text added: "Prog4"
- board text added: "RESET"
- board text added: "SWD"
- board text added: "SocketCan"
- board text added: "TERM"
- board text added: "TruckDevil"
- board text added: "VCC"
