File: CANTboard/CAN.sch (KiCad schematic (older format))
At the start: 15 parts, among them J3 Screw_Terminal_01x04, U4 MCP2558FD-xSN, U5 MCP2558FD-xSN, U6 74LVC1G66, U7 74LVC1G66

Commit message: Everything routed, commiting before last check before ordering PCBs
Parts:
- removed C16, C17, C18, C19: 100nF, Capacitor_SMD:C_0805_2012Metric, symbol Device:C
- added C16, C17, C18, C19: 100nF, Capacitor_SMD:C_0805_2012Metric, symbol Device:C_Small
Connections:
- net CAN1_H: now also J3.4 (Pin_4); no longer J3.2 (Pin_2)
- net CAN1_L: now also J3.3 (Pin_3); no longer J3.1 (Pin_1)
- net CAN3_H: now also J3.2 (Pin_2); no longer J3.4 (Pin_4)
- net CAN3_L: now also J3.1 (Pin_1); no longer J3.3 (Pin_3)
- net GND: now also C16.2, C17.1, C18.2, C19.1
- net VBUS: now also C17.2, C19.2
- net VCC: now also C16.1, C18.1
Changed lines of the file:
@@
 L power:GND #PWR?
 U 1 1 611CDDCF
-P 5050 3800
+P 4950 3800
 AR Path="/611CDDCF" Ref="#PWR?"  Part="1"
 AR Path="/611BBF4E/611CDDCF" Ref="#PWR038"  Part="1"
-F 0 "#PWR038" H 5050 3800 30  0001 C CNN
-F 1 "GND" H 5050 3730 30  0001 C CNN
-F 2 "" H 5050 3800 60  0000 C CNN
-F 3 "" H 5050 3800 60  0000 C CNN
-	1    5050 3800
+F 0 "#PWR038" H 4950 3800 30  0001 C CNN
+F 1 "GND" H 4950 3730 30  0001 C CNN
+F 2 "" H 4950 3800 60  0000 C CNN
+F 3 "" H 4950 3800 60  0000 C CNN
+	1    4950 3800
 	0    -1   -1   0
 $EndComp
@@
 L power:GND #PWR?
 U 1 1 611CDDDC
-P 3300 4800
+P 3300 4700
 AR Path="/611CDDDC" Ref="#PWR?"  Part="1"
 AR Path="/611BBF4E/611CDDDC" Ref="#PWR034"  Part="1"
-F 0 "#PWR034" H 3300 4800 30  0001 C CNN
-F 1 "GND" H 3300 4730 30  0001 C CNN
-F 2 "" H 3300 4800 60  0000 C CNN
-F 3 "" H 3300 4800 60  0000 C CNN
-	1    3300 4800
-	1    0    0    -1
-$EndComp
-Text GLabel 1100 1100 0    50   Input ~ 0
+F 0 "#PWR034" H 3300 4700 30  0001 C CNN
+F 1 "GND" H 3300 4630 30  0001 C CNN
+F 2 "" H 3300 4700 60  0000 C CNN
+F 3 "" H 3300 4700 60  0000 C CNN
+	1    3300 4700
+	1    0    0    -1
+$EndComp
+Text GLabel 1100 1300 0    50   Input ~ 0
 CAN1_L
-Text GLabel 1100 1200 0    50   Input ~ 0
+Text GLabel 1100 1400 0    50   Input ~ 0
 CAN1_H
 Text GLabel 4650 4300 2    50   Input ~ 0
@@
 Wire Wire Line
 	3300 4300 3650 4300
-Text GLabel 1100 1400 0    50   Input ~ 0
+Text GLabel 1100 1200 0    50   Input ~ 0
 CAN3_H
-Text GLabel 1100 1300 0    50   Input ~ 0
+Text GLabel 1100 1100 0    50   Input ~ 0
 CAN3_L
 $Comp
@@
 L power:GND #PWR?
 U 1 1 611CDE5F
-P 1050 4750
+P 1050 4650
 AR Path="/611CDE5F" Ref="#PWR?"  Part="1"
 AR Path="/611BBF4E/611CDE5F" Ref="#PWR028"  Part="1"
-F 0 "#PWR028" H 1050 4750 30  0001 C CNN
-F 1 "GND" H 1050 4680 30  0001 C CNN
-F 2 "" H 1050 4750 60  0000 C CNN
-F 3 "" H 1050 4750 60  0000 C CNN
-	1    1050 4750
+F 0 "#PWR028" H 1050 4650 30  0001 C CNN
+F 1 "GND" H 1050 4580 30  0001 C CNN
+F 2 "" H 1050 4650 60  0000 C CNN
+F 3 "" H 1050 4650 60  0000 C CNN
+	1    1050 4650
 	1    0    0    -1
 $EndComp
@@
 L power:GND #PWR?
 U 1 1 611CDE6B
-P 2750 3750
+P 2650 3750
 AR Path="/611CDE6B" Ref="#PWR?"  Part="1"
 AR Path="/611BBF4E/611CDE6B" Ref="#PWR032"  Part="1"
-F 0 "#PWR032" H 2750 3750 30  0001 C CNN
-F 1 "GND" H 2750 3680 30  0001 C CNN
-F 2 "" H 2750 3750 60  0000 C CNN
-F 3 "" H 2750 3750 60  0000 C CNN
-	1    2750 3750
+F 0 "#PWR032" H 2650 3750 30  0001 C CNN
+F 1 "GND" H 2650 3680 30  0001 C CNN
+F 2 "" H 2650 3750 60  0000 C CNN
+F 3 "" H 2650 3750 60  0000 C CNN
+	1    2650 3750
 	0    -1   -1   0
 $EndComp
@@
 	7500 1650 7500 1500
 Connection ~ 7500 1500
-$Comp
-L Device:C C?
-U 1 1 611CDE8A
-P 4900 3800
-AR Path="/611CDE8A" Ref="C?"  Part="1"
-AR Path="/611BBF4E/611CDE8A" Ref="C19"  Part="1"
-F 0 "C19" V 4648 3800 50  0000 C CNN
-F 1 "100nF" V 4739 3800 50  0000 C CNN
-F 2 "Capacitor_SMD:C_0805_2012Metric" H 4938 3650 50  0001 C CNN
-F 3 "~" H 4900 3800 50  0001 C CNN
-	1    4900 3800
-	0    1    1    0
-$EndComp
 Wire Wire Line
 	4150 3800 4600 3800
@@
 Wire Wire Line
 	4600 3800 4750 3800
-$Comp
-L Device:C C?
-U 1 1 611CDE93
-P 2600 3750
-AR Path="/611CDE93" Ref="C?"  Part="1"
-AR Path="/611BBF4E/611CDE93" Ref="C17"  Part="1"
-F 0 "C17" V 2348 3750 50  0000 C CNN
-F 1 "100nF" V 2439 3750 50  0000 C CNN
-F 2 "Capacitor_SMD:C_0805_2012Metric" H 2638 3600 50  0001 C CNN
-F 3 "~" H 2600 3750 50  0001 C CNN
-	1    2600 3750
-	0    1    1    0
-$EndComp
-$Comp
-L Device:C C?
-U 1 1 611CDE99
-P 1050 4600
-AR Path="/611CDE99" Ref="C?"  Part="1"
-AR Path="/611BBF4E/611CDE99" Ref="C16"  Part="1"
-F 0 "C16" H 935 4554 50  0000 R CNN
-F 1 "100nF" H 935 4645 50  0000 R CNN
-F 2 "Capacitor_SMD:C_0805_2012Metric" H 1088 4450 50  0001 C CNN
-F 3 "~" H 1050 4600 50  0001 C CNN
-	1    1050 4600
-	-1   0    0    1
-$EndComp
-$Comp
-L Device:C C?
-U 1 1 611CDE9F
-P 3300 4650
-AR Path="/611CDE9F" Ref="C?"  Part="1"
-AR Path="/611BBF4E/611CDE9F" Ref="C18"  Part="1"
-F 0 "C18" H 3185 4604 50  0000 R CNN
-F 1 "100nF" H 3185 4695 50  0000 R CNN
-F 2 "Capacitor_SMD:C_0805_2012Metric" H 3338 4500 50  0001 C CNN
-F 3 "~" H 3300 4650 50  0001 C CNN
-	1    3300 4650
-	-1   0    0    1
-$EndComp
 Wire Wire Line
 	1050 4450 1050 4250
@@
 Text Notes 6750 850  0    197  ~ 39
 Switches
+$Comp
+L Device:C_Small C16
+U 1 1 61334A14
+P 1050 4550
+F 0 "C16" H 1142 4596 50  0000 L CNN
+F 1 "100nF" H 1142 4505 50  0000 L CNN
+F 2 "Capacitor_SMD:C_0805_2012Metric" H 1050 4550 50  0001 C CNN
+F 3 "~" H 1050 4550 50  0001 C CNN
+	1    1050 4550
+	1    0    0    -1
+$EndComp
+$Comp
+L Device:C_Small C17
+U 1 1 613359EE
+P 2550 3750
+F 0 "C17" V 2321 3750 50  0000 C CNN
+F 1 "100nF" V 2412 3750 50  0000 C CNN
+F 2 "Capacitor_SMD:C_0805_2012Metric" H 2550 3750 50  0001 C CNN
+F 3 "~" H 2550 3750 50  0001 C CNN
+	1    2550 3750
+	0    1    1    0
+$EndComp
+$Comp
+L Device:C_Small C19
+U 1 1 613361C8
+P 4850 3800
+F 0 "C19" V 4621 3800 50  0000 C CNN
+F 1 "100nF" V 4712 3800 50  0000 C CNN
+F 2 "Capacitor_SMD:C_0805_2012Metric" H 4850 3800 50  0001 C CNN
+F 3 "~" H 4850 3800 50  0001 C CNN
+	1    4850 3800
+	0    1    1    0
+$EndComp
+$Comp
+L Device:C_Small C18
+U 1 1 61336920
+P 3300 4600
+F 0 "C18" H 3392 4646 50  0000 L CNN
+F 1 "100nF" H 3392 4555 50  0000 L CNN
+F 2 "Capacitor_SMD:C_0805_2012Metric" H 3300 4600 50  0001 C CNN
+F 3 "~" H 3300 4600 50  0001 C CNN
+	1    3300 4600
+	1    0    0    -1
+$EndComp
 $EndSCHEMATC
