File: CANTboard/USB.sch (KiCad schematic (older format))
At the start: 15 parts, among them J1 USB_C_Receptacle_USB2.0, U1 USB3343, U10 DSC1001

Commit message: Everything routed, commiting before last check before ordering PCBs
Parts:
- C25, C28, C29: value 0.1uF -> 100nF
Changed lines of the file:
@@
 P 4250 1150
 F 0 "C25" V 4479 1150 50  0000 C CNN
-F 1 "0.1uF" V 4388 1150 50  0000 C CNN
+F 1 "100nF" V 4388 1150 50  0000 C CNN
 F 2 "Capacitor_SMD:C_0805_2012Metric" H 4250 1150 50  0001 C CNN
 F 3 "~" H 4250 1150 50  0001 C CNN
@@
 P 5750 1500
 F 0 "C29" H 5842 1546 50  0000 L CNN
-F 1 "0.1uF" H 5842 1455 50  0000 L CNN
+F 1 "100nF" H 5842 1455 50  0000 L CNN
 F 2 "Capacitor_SMD:C_0805_2012Metric" H 5750 1500 50  0001 C CNN
 F 3 "~" H 5750 1500 50  0001 C CNN
@@
 P 2600 2900
 F 0 "C28" V 2371 2900 50  0000 C CNN
-F 1 "0.1uF" V 2462 2900 50  0000 C CNN
+F 1 "100nF" V 2462 2900 50  0000 C CNN
 F 2 "Capacitor_SMD:C_0805_2012Metric" H 2600 2900 50  0001 C CNN
 F 3 "~" H 2600 2900 50  0001 C CNN
