File: reCANT/J1708.sch (KiCad schematic (older format))
At the start: 11 parts, among them J4 Screw_Terminal_01x02, U8 SN74LVC1G14DBV, U9 ST485EBDR

Commit message: Add LCSC part numbers for each component. Not that chipocalypse makes building this right now feasible...
Parts:
- C20, C21: LCSC (none) -> C49678
- C22, C23: LCSC (none) -> C49217
- R12, R13: LCSC (none) -> C17673
- R14, R15: LCSC (none) -> C17714
- U8: LCSC (none) -> C7835
- U9: LCSC (none) -> C81186
Changed lines of the file:
@@
 F 2 "Package_SO:SOIC-8_3.9x4.9mm_P1.27mm" H 5100 2900 50  0001 C CNN
 F 3 "http://www.st.com/resource/en/datasheet/st485eb.pdf" H 5100 3850 50  0001 C CNN
+F 4 "C81186" H 5100 3800 50  0001 C CNN "LCSC"
 	1    5100 3800
 	1    0    0    -1
@@
 F 2 "Package_TO_SOT_SMD:SOT-23-5" H 4000 4050 50  0001 C CNN
 F 3 "http://www.ti.com/lit/ds/symlink/sn74lvc1g14.pdf" H 4000 4300 50  0001 C CNN
+F 4 "C7835" H 4000 4300 50  0001 C CNN "LCSC"
 	1    4000 4300
 	1    0    0    -1
@@
 F 3 "" H 5800 4400 30  0000 C CNN
 F 4 "MCR03ERTF1200" H 5800 4400 60  0001 C CNN "MPN"
+F 5 "C17673" V 5800 4400 50  0001 C CNN "LCSC"
 	1    5800 4400
 	-1   0    0    1
@@
 F 2 "Capacitor_SMD:C_0805_2012Metric" H 5838 3850 50  0001 C CNN
 F 3 "~" H 5800 4000 50  0001 C CNN
+F 4 "C49217" H 5800 4000 50  0001 C CNN "LCSC"
 	1    5800 4000
 	1    0    0    -1
@@
 F 2 "Capacitor_SMD:C_0805_2012Metric" H 5838 3550 50  0001 C CNN
 F 3 "~" H 5800 3700 50  0001 C CNN
+F 4 "C49217" H 5800 3700 50  0001 C CNN "LCSC"
 	1    5800 3700
 	1    0    0    -1
@@
 F 3 "" H 5800 3300 30  0000 C CNN
 F 4 "MCR03ERTF1200" H 5800 3300 60  0001 C CNN "MPN"
+F 5 "C17673" V 5800 3300 50  0001 C CNN "LCSC"
 	1    5800 3300
 	-1   0    0    1
@@
 F 3 "" H 6300 4300 30  0000 C CNN
 F 4 "MCR03ERTF1200" H 6300 4300 60  0001 C CNN "MPN"
+F 5 "C17714" V 6300 4300 50  0001 C CNN "LCSC"
 	1    6300 4300
 	0    -1   -1   0
@@
 F 3 "" H 6300 3550 30  0000 C CNN
 F 4 "MCR03ERTF1200" H 6300 3550 60  0001 C CNN "MPN"
+F 5 "C17714" V 6300 3550 50  0001 C CNN "LCSC"
 	1    6300 3550
 	0    -1   -1   0
@@
 F 2 "Capacitor_SMD:C_0805_2012Metric" H 4550 3400 50  0001 C CNN
 F 3 "~" H 4550 3400 50  0001 C CNN
+F 4 "C49678" H 4550 3400 50  0001 C CNN "LCSC"
 	1    4550 3400
 	0    -1   -1   0
@@
 F 2 "Capacitor_SMD:C_0805_2012Metric" H 3800 3950 50  0001 C CNN
 F 3 "~" H 3800 3950 50  0001 C CNN
+F 4 "C49678" H 3800 3950 50  0001 C CNN "LCSC"
 	1    3800 3950
 	0    -1   -1   0
