File: reCANT/LEDs.sch (KiCad schematic (older format))
At the start: 6 parts

Commit message: Add LCSC part numbers for each component. Not that chipocalypse makes building this right now feasible...
Parts:
- D1, D3: LCSC (none) -> C84256
- D2: LCSC (none) -> C2297
- R3, R4, R5: LCSC (none) -> C17802
Changed lines of the file:
@@
 F 3 "" H 2450 2400 30  0000 C CNN
 F 4 "MCR03ERTF1200" H 2450 2400 60  0001 C CNN "MPN"
+F 5 "C17802" V 2450 2400 50  0001 C CNN "LCSC"
 	1    2450 2400
 	-1   0    0    1
@@
 F 3 "" H 2450 2800 60  0000 C CNN
 F 4 "LTST-C191KRKT" H 2450 2800 60  0001 C CNN "MPN"
+F 5 "C84256" H 2450 2800 50  0001 C CNN "LCSC"
 	1    2450 2800
 	0    -1   -1   0
@@
 F 3 "" H 2000 2400 30  0000 C CNN
 F 4 "MCR03ERTF1200" H 2000 2400 60  0001 C CNN "MPN"
+F 5 "C17802" V 2000 2400 50  0001 C CNN "LCSC"
 	1    2000 2400
 	-1   0    0    1
@@
 F 3 "" H 1550 2400 30  0000 C CNN
 F 4 "MCR03ERTF1200" H 1550 2400 60  0001 C CNN "MPN"
+F 5 "C17802" V 1550 2400 50  0001 C CNN "LCSC"
 	1    1550 2400
 	-1   0    0    1
@@
 F 3 "" H 1550 2800 60  0000 C CNN
 F 4 "LTST-C191KRKT" H 1550 2800 60  0001 C CNN "MPN"
+F 5 "C84256" H 1550 2800 50  0001 C CNN "LCSC"
 	1    1550 2800
 	0    -1   -1   0
@@
 F 3 "" H 2000 2800 60  0000 C CNN
 F 4 "LTST-C191KGKT" H 2000 2800 60  0001 C CNN "MPN"
+F 5 "C2297" H 2000 2800 50  0001 C CNN "LCSC"
 	1    2000 2800
 	0    -1   -1   0
