File: reCANT_Teensy_Shield/reCANT_Teensy_Shield.kicad_pcb (KiCad board)
At the start: 2 copper layers, 90.3 x 20.8 mm, 45 parts, among them J1 Conn_02x08_Odd_Even, J2 Conn_01x24_Female, J3 Conn_01x24_Female, J4 Screw_Terminal_01x02, J5 Conn_01x03, J6 Screw_Terminal_01x04, J7 Screw_Terminal_01x02, J8 Conn_01x03, J9 Conn_01x03, U1 SN74LVC1G14DBV, U2 ST485EBDR, U3 MCP2558FD-xSN, U4 MCP2558FD-xSN, U5 MCP2558FD-xSN, U6 74LVC1G66, U7 74LVC1G66, U8 74LVC1G66

Commit message: Git silkscreen set
Parts:
- added G***: LOGO, Logo:logo, F.Cu at (76.8, 49.2)
Other:
- board text added: "+J1708-"
- board text added: "-CAN2+ -CAN1+"
- board text added: "CANT"
- board text added: "CanCat"
- board text added: "FD +CAN3-"
- board text added: "SocketCan"
- board text added: "TD"
- board text added: "reCANT Hat For Teensy 4.1 https://github.com/bitbane/CANT"
- board text added: "|TERM|"

Commit message: Added version number
Other:
- board text added: "reCANT Hat For Teensy 4.1 v0.1 https://github.com/bitbane/CANT"
- board text removed: "reCANT Hat For Teensy 4.1 https://github.com/bitbane/CANT"
Changed lines of the file:
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@@
     (effects (font (size 1 1) (thickness 0.15)))
   )
-  (gr_text "reCANT Hat For Teensy 4.1\nhttps://github.com/bitbane/CANT" (at 44.35 46.61) (layer "F.SilkS")
+  (gr_text "reCANT Hat For Teensy 4.1 v0.1\nhttps://github.com/bitbane/CANT" (at 44.35 46.61) (layer "F.SilkS")
     (effects (font (size 1 1) (thickness 0.15)))
   )
